File: kicad/eink-audio-player.kicad_sch (KiCad schematic)
At the start: 18 parts, among them J1 Feather 16-pin, J10 TLV MICBIAS..MIC, J2 Feather 12-pin, J4 EYESPI 1-9 (5613 JP2), J5 EYESPI 10-18 (5613 JP1), J9 TLV VIN..SPKP, SW1 Power (MSK-12C03)

Commit message: Add TP1-TP2 jumper pads for a D5 to TLV MCLK wire
Two 3.8 x 2.0 mm SMD pads: TP1 on Feather D5, TP2 on TLV320 MCLK, with
silkscreen and a schematic note. A 15 MHz PWM clock on D5 lets the TLV
PLL lock; running it from BCLK sounds muffled. DRC: no new errors.

Co-Authored-By: Claude Opus 5.5 (1M context) <noreply@anthropic.com>
Parts:
- added TP1, TP2: JUMPER, eink-audio-player:JumperPad_3.8x2.0mm, symbol Connector:TestPoint
Connections:
- net D5_MCLK_JMP: now reaches J2.10 (Pin_10)
- net D5_MCLK_JMP: now also TP1.1
- net MCLK: now reaches J9.8 (Pin_8)
- net MCLK: now also TP2.1
- no-connect marks 32 -> 30
Other:
- note added: "JUMPER WIRE: solder TP1 (Feather D5) to TP2 (TLV MCLK)"
- note added: "MCLK: D5 drives a 15 MHz PWM clock (pwmio, configure_clocks mclk_freq=15_000_000). With BCLK only, the TLV PLL does not lock and audio sounds muffled."
- note added: "TLV RST (J10.5) open: 10K pull-up on the breakout. MCLK on TP2, wired to D5 on TP1."
- note removed: "TLV RST (J10.5) open: 10K pull-up on the breakout. MCLK open: PLL from BCLK."
Changed lines of the file:
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@@
 	(no_connect (at 55.88 144.78))
 	(no_connect (at 55.88 147.32))
-	(no_connect (at 55.88 149.86))
+	(wire (pts (xy 55.88 149.86) (xy 50.8 149.86))
+		(stroke (width 0) (type default)))
+	(label "D5_MCLK_JMP" (at 50.8 149.86 180) (fields_autoplaced yes)
+		(effects (font (size 1.27 1.27)) (justify right bottom))
+)
 	(wire (pts (xy 55.88 152.4) (xy 50.8 152.4))
 		(stroke (width 0) (type default)))
@@
 		(effects (font (size 1.27 1.27)) (justify right bottom))
 )
-	(no_connect (at 127.0 83.82))
+	(wire (pts (xy 127.0 83.82) (xy 121.92 83.82))
+		(stroke (width 0) (type default)))
+	(label "MCLK" (at 121.92 83.82 180) (fields_autoplaced yes)
+		(effects (font (size 1.27 1.27)) (justify right bottom))
+)
 	(no_connect (at 127.0 86.36))
 	(no_connect (at 127.0 88.9))
@@
 		(effects (font (size 1.27 1.27)) (justify left bottom))
 )
-	(text "TLV RST (J10.5) open: 10K pull-up on the breakout. MCLK open: PLL from BCLK." (exclude_from_sim no) (at 30.48 187.96 0)
-		(effects (font (size 1.27 1.27)) (justify left bottom))
-)
+	(text "TLV RST (J10.5) open: 10K pull-up on the breakout. MCLK on TP2, wired to D5 on TP1." (exclude_from_sim no) (at 30.48 187.96 0)
+		(effects (font (size 1.27 1.27)) (justify left bottom))
+)
+	(symbol (lib_id "Connector:TestPoint") (at 110.49 167.64 0) (unit 1)
+		(exclude_from_sim no) (in_bom no) (on_board yes) (dnp no)
+		(property "Reference" "TP1" (at 110.49 160.782 0)
+			(effects (font (size 1.27 1.27)))
+		)
+		(property "Value" "JUMPER" (at 110.49 162.56 0)
+			(effects (font (size 1.27 1.27)))
+		)
+		(property "Footprint" "eink-audio-player:JumperPad_3.8x2.0mm" (at 110.49 167.64 0)
+			(effects (font (size 1.27 1.27)) (hide yes))
+		)
+		(property "Datasheet" "~" (at 110.49 167.64 0)
+			(effects (font (size 1.27 1.27)) (hide yes))
+		)
+		(pin "1")
+		(instances (project "eink-audio-player"
+			(path "/68a20767-e11b-5af4-a54e-061cf37f3ec1" (reference "TP1") (unit 1))))
+	)
+	(wire (pts (xy 110.49 167.64) (xy 102.87 167.64))
+		(stroke (width 0) (type default)))
+	(label "D5_MCLK_JMP" (at 102.87 167.64 180) (fields_autoplaced yes)
+		(effects (font (size 1.27 1.27)) (justify right bottom))
+)
+	(symbol (lib_id "Connector:TestPoint") (at 156.21 167.64 0) (unit 1)
+		(exclude_from_sim no) (in_bom no) (on_board yes) (dnp no)
+		(property "Reference" "TP2" (at 156.21 160.782 0)
+			(effects (font (size 1.27 1.27)))
+		)
+		(property "Value" "JUMPER" (at 156.21 162.56 0)
+			(effects (font (size 1.27 1.27)))
+		)
+		(property "Footprint" "eink-audio-player:JumperPad_3.8x2.0mm" (at 156.21 167.64 0)
+			(effects (font (size 1.27 1.27)) (hide yes))
+		)
+		(property "Datasheet" "~" (at 156.21 167.64 0)
+			(effects (font (size 1.27 1.27)) (hide yes))
+		)
+		(pin "1")
+		(instances (project "eink-audio-player"
+			(path "/68a20767-e11b-5af4-a54e-061cf37f3ec1" (reference "TP2") (unit 1))))
+	)
+	(wire (pts (xy 156.21 167.64) (xy 148.59 167.64))
+		(stroke (width 0) (type default)))
+	(label "MCLK" (at 148.59 167.64 180) (fields_autoplaced yes)
+		(effects (font (size 1.27 1.27)) (justify right bottom))
+)
+	(text "JUMPER WIRE: solder TP1 (Feather D5) to TP2 (TLV MCLK)" (exclude_from_sim no) (at 100.33 158.75 0)
+		(effects (font (size 1.524 1.524) bold) (justify left bottom))
+)
+	(text "MCLK: D5 drives a 15 MHz PWM clock (pwmio, configure_clocks mclk_freq=15_000_000). With BCLK only, the TLV PLL does not lock and audio sounds muffled." (exclude_from_sim no) (at 30.48 193.04 0)
+		(effects (font (size 1.27 1.27)) (justify left bottom))
+)
