File: kicad/frisson.kicad_pcb (KiCad board)
At the start: 2 copper layers, 76.1 x 61 mm, 27 parts, among them J1 Feather 16-pin, J10 TLV MICBIAS..MIC, J2 Feather 12-pin, J4 EYESPI 1-9 (5613 JP2), J5 EYESPI 10-18 (5613 JP1), J9 TLV VIN..SPKP, SW1 Power (MSK-12C03)

Commit message: Rename files from eink-audio-player to frisson
Co-Authored-By: Claude Opus 5.5 (1M context) <noreply@anthropic.com>
Parts:
- SW1: footprint eink-audio-player:SW_SPDT_MSK-12C03 -> frisson:SW_SPDT_MSK-12C03
- TP1, TP2: footprint eink-audio-player:JumperPad_3.8x2.0mm -> frisson:JumperPad_3.8x2.0mm
Changed lines of the file:
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@@
 		)
 	)
-	(footprint "eink-audio-player:JumperPad_3.8x2.0mm"
+	(footprint "frisson:JumperPad_3.8x2.0mm"
 		(layer "F.Cu")
 		(at 120 89.91)
@@
 		(embedded_fonts no)
 	)
-	(footprint "eink-audio-player:SW_SPDT_MSK-12C03"
+	(footprint "frisson:SW_SPDT_MSK-12C03"
 		(layer "F.Cu")
 		(at 97.78 79.59 180)
@@
 		)
 	)
-	(footprint "eink-audio-player:JumperPad_3.8x2.0mm"
+	(footprint "frisson:JumperPad_3.8x2.0mm"
 		(layer "F.Cu")
 		(at 107.6 116.91)
