File: kicad/frisson.kicad_sch (KiCad schematic)
At the start: 20 parts, among them J1 Feather 16-pin, J10 TLV MICBIAS..MIC, J2 Feather 12-pin, J4 EYESPI 1-9 (5613 JP2), J5 EYESPI 10-18 (5613 JP1), J9 TLV VIN..SPKP, SW1 Power (MSK-12C03)

Commit message: Rename files from eink-audio-player to frisson
Co-Authored-By: Claude Opus 5.5 (1M context) <noreply@anthropic.com>
Parts:
- SW1: footprint eink-audio-player:SW_SPDT_MSK-12C03 -> frisson:SW_SPDT_MSK-12C03
- TP1, TP2: footprint eink-audio-player:JumperPad_3.8x2.0mm -> frisson:JumperPad_3.8x2.0mm
Other:
- title: eink-audio-player -> frisson
Changed lines of the file:
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@@
 	(generator_version "8.0")
 	(paper "A3")
-	(title_block (title "eink-audio-player") (company "mikeysklar"))
+	(title_block (title "frisson") (company "mikeysklar"))
 	(symbol (lib_id "Connector:Conn_01x16_Socket") (at 60.96 76.2 0) (unit 1)
 		(exclude_from_sim no) (in_bom yes) (on_board yes) (dnp no)
@@
 		(pin "15")
 		(pin "16")
-		(instances (project "eink-audio-player"
+		(instances (project "frisson"
 			(path "/68a20767-e11b-5af4-a54e-061cf37f3ec1" (reference "J1") (unit 1))))
 	)
@@
 		(pin "11")
 		(pin "12")
-		(instances (project "eink-audio-player"
+		(instances (project "frisson"
 			(path "/68a20767-e11b-5af4-a54e-061cf37f3ec1" (reference "J2") (unit 1))))
 	)
@@
 		(pin "9")
 		(pin "10")
-		(instances (project "eink-audio-player"
+		(instances (project "frisson"
 			(path "/68a20767-e11b-5af4-a54e-061cf37f3ec1" (reference "J9") (unit 1))))
 	)
@@
 		(pin "7")
 		(pin "8")
-		(instances (project "eink-audio-player"
+		(instances (project "frisson"
 			(path "/68a20767-e11b-5af4-a54e-061cf37f3ec1" (reference "J10") (unit 1))))
 	)
@@
 		(pin "8")
 		(pin "9")
-		(instances (project "eink-audio-player"
+		(instances (project "frisson"
 			(path "/68a20767-e11b-5af4-a54e-061cf37f3ec1" (reference "J4") (unit 1))))
 	)
@@
 		(pin "8")
 		(pin "9")
-		(instances (project "eink-audio-player"
+		(instances (project "frisson"
 			(path "/68a20767-e11b-5af4-a54e-061cf37f3ec1" (reference "J5") (unit 1))))
 	)
@@
 			(effects (font (size 1.27 1.27)))
 		)
-		(property "Footprint" "eink-audio-player:SW_SPDT_MSK-12C03" (at 203.2 139.7 0)
+		(property "Footprint" "frisson:SW_SPDT_MSK-12C03" (at 203.2 139.7 0)
 			(effects (font (size 1.27 1.27)) (hide yes))
 		)
@@
 		(pin "2")
 		(pin "3")
-		(instances (project "eink-audio-player"
+		(instances (project "frisson"
 			(path "/68a20767-e11b-5af4-a54e-061cf37f3ec1" (reference "SW1") (unit 1))))
 	)
@@
 		(pin "1")
 		(pin "2")
-		(instances (project "eink-audio-player"
+		(instances (project "frisson"
 			(path "/68a20767-e11b-5af4-a54e-061cf37f3ec1" (reference "R1") (unit 1))))
 	)
@@
 		(pin "1")
 		(pin "2")
-		(instances (project "eink-audio-player"
+		(instances (project "frisson"
 			(path "/68a20767-e11b-5af4-a54e-061cf37f3ec1" (reference "R2") (unit 1))))
 	)
@@
 		(pin "1")
 		(pin "2")
-		(instances (project "eink-audio-player"
+		(instances (project "frisson"
 			(path "/68a20767-e11b-5af4-a54e-061cf37f3ec1" (reference "R3") (unit 1))))
 	)
@@
 		(pin "1")
 		(pin "2")
-		(instances (project "eink-audio-player"
+		(instances (project "frisson"
 			(path "/68a20767-e11b-5af4-a54e-061cf37f3ec1" (reference "R4") (unit 1))))
 	)
@@
 			(effects (font (size 1.27 1.27)) (hide yes))
 		)
-		(instances (project "eink-audio-player"
+		(instances (project "frisson"
 			(path "/68a20767-e11b-5af4-a54e-061cf37f3ec1" (reference "H1") (unit 1))))
 	)
@@
 			(effects (font (size 1.27 1.27)) (hide yes))
 		)
-		(instances (project "eink-audio-player"
+		(instances (project "frisson"
 			(path "/68a20767-e11b-5af4-a54e-061cf37f3ec1" (reference "H2") (unit 1))))
 	)
@@
 			(effects (font (size 1.27 1.27)) (hide yes))
 		)
-		(instances (project "eink-audio-player"
+		(instances (project "frisson"
 			(path "/68a20767-e11b-5af4-a54e-061cf37f3ec1" (reference "H3") (unit 1))))
 	)
@@
 			(effects (font (size 1.27 1.27)) (hide yes))
 		)
-		(instances (project "eink-audio-player"
+		(instances (project "frisson"
 			(path "/68a20767-e11b-5af4-a54e-061cf37f3ec1" (reference "H4") (unit 1))))
 	)
@@
 			(effects (font (size 1.27 1.27)) (hide yes))
 		)
-		(instances (project "eink-audio-player"
+		(instances (project "frisson"
 			(path "/68a20767-e11b-5af4-a54e-061cf37f3ec1" (reference "H5") (unit 1))))
 	)
@@
 			(effects (font (size 1.27 1.27)) (hide yes))
 		)
-		(instances (project "eink-audio-player"
+		(instances (project "frisson"
 			(path "/68a20767-e11b-5af4-a54e-061cf37f3ec1" (reference "H6") (unit 1))))
 	)
@@
 			(effects (font (size 1.27 1.27)) (hide yes))
 		)
-		(instances (project "eink-audio-player"
+		(instances (project "frisson"
 			(path "/68a20767-e11b-5af4-a54e-061cf37f3ec1" (reference "H7") (unit 1))))
 	)
@@
 			(effects (font (size 1.27 1.27)))
 		)
-		(property "Footprint" "eink-audio-player:JumperPad_3.8x2.0mm" (at 110.49 167.64 0)
+		(property "Footprint" "frisson:JumperPad_3.8x2.0mm" (at 110.49 167.64 0)
 			(effects (font (size 1.27 1.27)) (hide yes))
 		)
@@
 		)
 		(pin "1")
-		(instances (project "eink-audio-player"
+		(instances (project "frisson"
 			(path "/68a20767-e11b-5af4-a54e-061cf37f3ec1" (reference "TP1") (unit 1))))
 	)
@@
 			(effects (font (size 1.27 1.27)))
 		)
-		(property "Footprint" "eink-audio-player:JumperPad_3.8x2.0mm" (at 156.21 167.64 0)
+		(property "Footprint" "frisson:JumperPad_3.8x2.0mm" (at 156.21 167.64 0)
 			(effects (font (size 1.27 1.27)) (hide yes))
 		)
@@
 		)
 		(pin "1")
-		(instances (project "eink-audio-player"
+		(instances (project "frisson"
 			(path "/68a20767-e11b-5af4-a54e-061cf37f3ec1" (reference "TP2") (unit 1))))
 	)
